Commit message: scaffolded further ROS architecture and stubbed interfaces

File: src/g1_description/g1_23dof.urdf.xacro (robot description, xacro)
@@ -12,4 +12,15 @@
   -->
   <xacro:arg name="hardware_plugin" default="mujoco_ros2_control/MujocoSystem"/>
+  <!-- REP-105 root frame. The Unitree model's own root link is `pelvis`; this
+       massless `base_link` + fixed identity joint is added so the TF contract
+       (odom -> base_link, see INTERFACE_CONTRACT.md) and Nav2's default
+       robot_base_frame work without renaming anything. No geometry/inertia is
+       affected. -->
+  <link name="base_link"/>
+  <joint name="base_link_to_pelvis" type="fixed">
+    <parent link="base_link"/>
+    <child link="pelvis"/>
+    <origin xyz="0 0 0" rpy="0 0 0"/>
+  </joint>
   <material name="dark">
     <color rgba="0.2 0.2 0.2 1"/>
@@ -853,5 +864,5 @@
   <ros2_control name="G1System" type="system">
     <hardware>
-      <plugin>${hardware_plugin}</plugin>
+      <plugin>$(arg hardware_plugin)</plugin>
       <!-- Consumed only by ethercat_bridge/EthercatHardwareInterface (ignored by
            mujoco_ros2_control/MujocoSystem, which does not look up these keys).
